File: schematic/pcb/pcb.kicad_pcb (KiCad board)
At the start: 4 copper layers, 90 x 69 mm, 40 parts, among them J1 MAVLINK, J2 DISPLAY, J3 SER. SERVO, J4 MAG., J5 SERVO, J6 5V, P1 USB_C_Plug_USB2.0, Q1 NPN, Q2 NPN, SW1 SW_Push, SW2 SW_Push, SW3 SW_Push, SW4 SW_Push, SW5 SW_Push, SW6 SW_Push

Commit message: v. alpha pcb 2
Parts:
- added G***: LOGO, LOGO, F.Cu at (174.3, 81.1)
- renumbered SW3 to SW1, SW4 to SW2, SW5 to SW3, SW6 to SW4
Routing:
- net IO0: track 94.9 -> 96.2 mm
- net DTR: track 12.5 -> 11.9 mm
Other:
- board text added: "."
- board text added: "3V3"
- board text added: "SDI"
- board text added: "v. alpha 4/2024"

Commit message: pcb v3
Parts:
- added D1: POWER, LED_SMD:LED_0805_2012Metric, F.Cu at (106.1, 106.3)
- added D2: TX, LED_SMD:LED_0805_2012Metric, F.Cu at (123.1, 79.3)
- added D3: RX, LED_SMD:LED_0805_2012Metric, F.Cu at (123.1, 81.5)
- added R10: 5K, Resistor_SMD:R_0805_2012Metric, F.Cu at (126.8, 81.5)
- added R8: 5K, Resistor_SMD:R_0805_2012Metric, F.Cu at (109.7, 106.3)
- added R9: 5K, Resistor_SMD:R_0805_2012Metric, F.Cu at (126.8, 79.3)
- LDO1: renamed from 3V3 LDO
- SW1: value SW_Push -> BOOT
- SW2: value SW_Push -> RESET
- moved G*** 69.1 mm to (115.0, 116.5), turned to 0 degrees
- moved ? 66.3 mm to (187.2, 126.5)
- moved ? 66.3 mm to (107.2, 126.5)
- moved C1 66.3 mm to (116.3, 80.3)
- moved C2 66.3 mm to (108.3, 80.3)
- moved C4 66.3 mm to (119.0, 99.2)
- moved C5 66.3 mm to (119.0, 97.0)
- moved C9 66.3 mm to (128.6, 71.7)
- moved CP1 66.3 mm to (124.2, 95.5)
- moved ESP1 66.3 mm to (148.3, 72.1)
- moved J1 66.3 mm to (187.8, 112.2)
- moved J2 66.3 mm to (187.8, 100.3)
- moved J6 66.3 mm to (165.7, 66.3)
- moved P1 66.3 mm to (106.2, 95.5)
- moved R3 66.3 mm to (123.3, 103.1)
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- renumbered ANTENNA to C3, ESP32 to ESP1, SW1 to SW3, SW2 to SW4, SW3 to SW5, SW4 to SW6, GPS to U1
Routing:
- net ESP32_RX0: track 47.7 -> 56.7 mm, vias 2 -> 3
- net ESP32_TX0: track 51.6 -> 59.2 mm, vias 2 -> 3
- net +3V3: track 30.1 -> 35.0 mm, vias 7 -> 9
- net Net-(D3-K): track 0.00 -> 1.89 mm
- net Net-(D2-K): track 0.00 -> 1.85 mm
- net Net-(D1-A): track 0.00 -> 1.76 mm
- added copper zone on B.Cu, net GND
Other:
- board text added: "ANTENNA"
- board text added: "BOOT"
- board text added: "ESP32 WROOM 32"
- board text added: "GPS"
- board text added: "POWER"
- board text added: "RESET"

Commit message: added leds
Parts:
- moved G*** 1.50 mm to (116.5, 116.5)
Routing:
- net BUTTON_2: track 156.7 -> 54.0 mm
- net BUTTON_1: track 143.9 -> 59.2 mm
- net IO0: track 96.2 -> 73.8 mm
- net EN: track 61.9 -> 48.5 mm, vias 2 -> 0
- net GND: track 83.5 -> 91.9 mm
- net BUTTON_4: track 82.9 -> 79.3 mm
- net GPS_SCK: track 44.7 -> 45.6 mm
- net GPS_MISO: track 42.1 -> 42.8 mm
- net MAV_RX: track 80.7 -> 80.1 mm
- net MAV_TX: track 83.2 -> 82.6 mm

Commit message: pcb final v1
Parts:
- added C11: 10uF, Capacitor_SMD:C_0805_2012Metric, F.Cu at (172.0, 84.1)
- added C12: 0.1uF, Capacitor_SMD:C_0805_2012Metric, F.Cu at (174.1, 84.1)
- added REF**: OSHW-Logo_38.1x40mm_SilkScreen, Symbol:OSHW-Logo_38.1x40mm_SilkScreen, B.Cu at (147.8, 100.7)
- C5: value 4.7uF -> 10uF
- R1, R2: value 10K 5% -> 10K
- R5: value 2K 5% -> 2K
- R6: value 10K 5% (NC) -> 10K (NC)
- moved G*** 0.85 mm to (116.2, 117.3)
Routing:
- net +3V3: track 35.0 -> 41.9 mm
- net +5V: track 181.0 -> 175.7 mm
- net DTR: track 11.9 -> 12.5 mm
- net SERVO: vias 0 -> 1
- net GND: vias 60 -> 86
Other:
- board text added: "BUTTON 1"
- board text added: "BUTTON 2"
- board text added: "BUTTON 3"
- board text added: "BUTTON 4"
- board text added: "NC"
- board text added: "TRACKER PCB v. alpha 4/2024"
- board text added: "{ "ViaStitching": "0.2", "stitch_zone_0": { "HSpacing": "1", "VSpacing": "1", "Clearance": "0", "Randomize": false } }"
- board text removed: "v. alpha 4/2024"

Commit message: gps tweaks
Other:
- board text removed: "{ "ViaStitching": "0.2", "stitch_zone_0": { "HSpacing": "1", "VSpacing": "1", "Clearance": "0", "Randomize": false } }"
