File: schematic/pcb/_autosave-pcb.kicad_pcb (KiCad board)
At the start: 4 copper layers, 90 x 69 mm, 40 parts, among them J1 MAVLINK, J2 DISPLAY, J3 SER. SERVO, J4 MAG., J5 SERVO, J6 5V, P1 USB_C_Plug_USB2.0, Q1 NPN, Q2 NPN, SW1 SW_Push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

Commit message: v. alpha pcb
Parts:
- renumbered SW3 to SW1, SW4 to SW2, SW5 to SW3, SW6 to SW4
Routing:
- net IO0: track 94.9 -> 96.2 mm
- net DTR: track 12.5 -> 11.9 mm
Other:
- board text added: "."
- board text added: "3V3"
- board text added: "SDI"
- board text added: "v. alpha 4/2024"
