File: schematic/pcb/pcb.kicad_sch (KiCad schematic)
At the start: 32 parts, among them J1 MAVLINK, J2 DISPLAY, J3 SER. SERVO, J4 MAG., J5 SERVO, J6 5V, P1 USB_C_Plug_USB2.0, Q1 NPN, Q2 NPN, SW1 SW_Push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

Commit message: trzymam kciuki
Parts:
- J6: footprint Connector_Wuerth:Wuerth_WR-WTB_64800211622_1x02_P1.50mm_Vertical -> Connector_Amphenol:VI0221550000G
- P1: footprint Connector_USB:USB_C_Receptacle_GCT_USB4135-GF-A_6P_TopMnt_Horizontal -> Connector_USB:USB_C_Receptacle_HRO_TYPE-C-31-M-12
Connections:
- net +5V: now also J6.2 (Pin_2); no longer J6.1 (Pin_1)
- net GND: now also J6.1 (Pin_1); no longer J6.2 (Pin_2)
Changed lines of the file:
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@@
-    (stroke (width 0) (type default))
-  )
-  (wire (pts (xy 206.375 151.765) (xy 203.2 151.765))
     (stroke (width 0) (type default))
   )
@@
   )
   (wire (pts (xy 186.055 102.87) (xy 181.61 102.87))
+    (stroke (width 0) (type default))
+  )
+  (wire (pts (xy 206.375 154.305) (xy 203.2 154.305))
     (stroke (width 0) (type default))
   )
@@
     (stroke (width 0) (type default))
   )
-  (wire (pts (xy 206.375 149.225) (xy 206.375 151.765))
+  (wire (pts (xy 206.375 149.225) (xy 206.375 154.305))
     (stroke (width 0) (type default))
   )
@@
     (stroke (width 0) (type default))
   )
-  (wire (pts (xy 206.375 154.305) (xy 206.375 156.21))
-    (stroke (width 0) (type default))
-  )
   (wire (pts (xy 27.305 100.965) (xy 30.48 100.965))
     (stroke (width 0) (type default))
@@
     (stroke (width 0) (type default))
   )
+  (wire (pts (xy 207.645 151.765) (xy 203.2 151.765))
+    (stroke (width 0) (type default))
+  )
   (wire (pts (xy 120.015 170.815) (xy 120.015 172.085))
     (stroke (width 0) (type default))
@@
     (stroke (width 0) (type default))
   )
+  (wire (pts (xy 207.645 156.21) (xy 207.645 151.765))
+    (stroke (width 0) (type default))
+  )
   (wire (pts (xy 100.33 64.77) (xy 100.33 67.31))
     (stroke (width 0) (type default))
@@
   )
   (wire (pts (xy 45.72 76.2) (xy 45.72 78.105))
-    (stroke (width 0) (type default))
-  )
-  (wire (pts (xy 203.2 154.305) (xy 206.375 154.305))
     (stroke (width 0) (type default))
   )
@@
       (effects (font (size 1.27 1.27)))
     )
-    (property "Footprint" "Connector_USB:USB_C_Receptacle_GCT_USB4135-GF-A_6P_TopMnt_Horizontal" (at 131.445 147.955 0)
+    (property "Footprint" "Connector_USB:USB_C_Receptacle_HRO_TYPE-C-31-M-12" (at 131.445 147.955 0)
       (effects (font (size 1.27 1.27)) hide)
     )
@@
       (effects (font (size 1.27 1.27)))
     )
-    (property "Footprint" "Connector_Wuerth:Wuerth_WR-WTB_64800211622_1x02_P1.50mm_Vertical" (at 198.12 151.765 0)
+    (property "Footprint" "Connector_Amphenol:VI0221550000G" (at 198.12 151.765 0)
       (effects (font (size 1.27 1.27)) hide)
     )
@@
     )
   )
-  (symbol (lib_id "power:GND") (at 206.375 156.21 0) (unit 1)
-    (in_bom yes) (on_board yes) (dnp no) (fields_autoplaced)
-    (property "Reference" "#PWR024" (at 206.375 162.56 0)
-      (effects (font (size 1.27 1.27)) hide)
-    )
-    (property "Value" "GND" (at 206.375 160.528 0)
-      (effects (font (size 1.27 1.27)))
-    )
-    (property "Footprint" "" (at 206.375 156.21 0)
-      (effects (font (size 1.27 1.27)) hide)
-    )
-    (property "Datasheet" "" (at 206.375 156.21 0)
-      (effects (font (size 1.27 1.27)) hide)
-    )
+  (symbol (lib_id "power:GND") (at 207.645 156.21 0) (unit 1)
+    (in_bom yes) (on_board yes) (dnp no) (fields_autoplaced)
+    (property "Reference" "#PWR024" (at 207.645 162.56 0)
+      (effects (font (size 1.27 1.27)) hide)
+    )
+    (property "Value" "GND" (at 207.645 160.528 0)
+      (effects (font (size 1.27 1.27)))
+    )
+    (property "Footprint" "" (at 207.645 156.21 0)
+      (effects (font (size 1.27 1.27)) hide)
+    )
+    (property "Datasheet" "" (at 207.645 156.21 0)
+      (effects (font (size 1.27 1.27)) hide)
+    )

Commit message: lets go
Parts:
- ESP1: footprint RF_Module:ESP32-WROOM-32 -> RF_Module:ESP32-WROOM-32U
Changed lines of the file:
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@@
       (effects (font (size 1.27 1.27)) (justify left))
     )
-    (property "Footprint" "RF_Module:ESP32-WROOM-32" (at 236.855 109.22 0)
+    (property "Footprint" "RF_Module:ESP32-WROOM-32U" (at 236.855 109.22 0)
       (effects (font (size 1.27 1.27)) hide)
     )

Commit message: new pcb
Parts:
- removed J3: SER. SERVO, Connector_JST:JST_GH_BM04B-GHS-TBT_1x04-1MP_P1.25mm_Vertical, symbol Connector:Conn_01x04_Pin
- added J3: SER. SERVO, Connector_JST:JST_GH_BM03B-GHS-TBT_1x03-1MP_P1.25mm_Vertical, symbol Connector:Conn_01x03_Pin
- added SW3, SW4, SW5, SW6: SW_Push, Button_Switch_SMD:SW_SPST_B3SL-1002P, symbol Switch:SW_Push
- ESP1: footprint RF_Module:ESP32-WROOM-32U -> RF_Module:ESP32-WROOM-32
- J6: footprint Connector_Amphenol:VI0221550000G -> Connector_PinHeader_2.54mm:PinHeader_1x02_P2.54mm_Vertical
- SW1, SW2: footprint (none) -> Button_Switch_SMD:SW_SPST_B3U-1000P
Connections:
- net +3V3: now also J4.1 (Pin_1)
- net +5V: now also J1.1 (Pin_1), J2.1 (Pin_1)
- net GND: now also J1.2 (Pin_2), J2.2 (Pin_2), J4.2 (Pin_2), J3.1 (Pin_1), SW3.1, SW4.1, SW5.1, SW6.1
- net SCREEN_CS: now also J2.5 (Pin_5)
- net SCREEN_MOSI: now also J2.4 (Pin_4)
- net SCREEN_SCK: now also J2.3 (Pin_3)
- net MAV_RX: now reaches J1.3 (Pin_3)
- net MAV_RX: now also ESP1.9 (IO33)
- net MAV_TX: now reaches J1.4 (Pin_4)
- net MAV_TX: now also ESP1.8 (IO32)
- net SERVO: now reaches J5.2 (Pin_2)
- net SERVO: now also ESP1.26 (IO4)
- net MAG_SDI: now reaches J4.3 (Pin_3)
- net MAG_SDI: now also ESP1.33 (IO21)
- net MAG_SCK: now reaches J4.4 (Pin_4)
- net MAG_SCK: now also ESP1.36 (IO22)
- net BUTTON_1: now reaches ESP1.10 (IO25)
- net BUTTON_1: now also SW3.2
- net BUTTON_2: now reaches ESP1.11 (IO26)
- net BUTTON_2: now also SW4.2
- net SERVO_RX: now reaches ESP1.27 (IO16)
- net SERVO_RX: now also J3.2 (Pin_2)
- net SERVO_TX: now reaches ESP1.28 (IO17)
- net SERVO_TX: now also J3.3 (Pin_3)
- net BUTTON_3: now reaches ESP1.6 (IO34)
- net BUTTON_3: now also SW5.2
- net BUTTON_4: now reaches ESP1.7 (IO35)
- net BUTTON_4: now also SW6.2
Other:
- moved on the sheet: C8, C9, J1, J2, J4, J5, J6, P1, Q1, Q2, R1, R2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

Commit message: v. alpha pcb
Connections:
- no-connect marks 22 -> 23
Changed lines of the file:
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@@
   (no_connect (at 30.48 113.665))
   (no_connect (at 141.605 90.805))
+  (no_connect (at 254.635 73.66))
   (no_connect (at 141.605 85.725))
   (no_connect (at 141.605 80.645))

Commit message: pcb v3
Parts:
- added D1: POWER, LED_SMD:LED_0805_2012Metric, symbol Device:LED_Small
- added D2: TX, LED_SMD:LED_0805_2012Metric, symbol Device:LED_Small
- added D3: RX, LED_SMD:LED_0805_2012Metric, symbol Device:LED_Small
- added R10, R8, R9: 5K, Resistor_SMD:R_0805_2012Metric, symbol Device:R_Small
- SW1: value SW_Push -> BOOT
- SW2: value SW_Push -> RESET
Connections:
- net +3V3: now also D2.2 (A), D3.2 (A), R8.1
- net ESP32_RX0: now also R10.1
- net ESP32_TX0: now also R9.2
- net GND: now also D1.1 (K)
- new net: D2.1 (K), R9.1
- new net: D1.2 (A), R8.2
- new net: D3.1 (K), R10.2
Other:
- moved on the sheet: C7, R7
