File: schematic/pcb/pcb.kicad_sch (KiCad schematic)
At the start: 44 parts, among them J1 MAVLINK, J2 DISPLAY, J3 SER. SERVO, J4 MAG., J5 SERVO, J6 5V, P1 USB_C_Plug_USB2.0, Q1 NPN, Q2 NPN, SW1 BOOT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

Commit message: inventor model, geotransform coeff param
Parts:
- R1, R2: value 10K 5% -> 10K
- R5: value 2K -> 5K
Changed lines of the file:
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@@
   (symbol (lib_id "Device:R_Small") (at 35.56 160.655 270) (unit 1)
     (in_bom yes) (on_board yes) (dnp no) (fields_autoplaced)
-    (property "Reference" "R2" (at 35.56 155.575 90)
-      (effects (font (size 1.27 1.27)))
-    )
-    (property "Value" "10K 5%" (at 35.56 158.115 90)
+    (property "Reference" "R2" (at 35.56 154.94 90)
+      (effects (font (size 1.27 1.27)))
+    )
+    (property "Value" "10K" (at 35.56 157.48 90)
       (effects (font (size 1.27 1.27)))
     )
@@
       (effects (font (size 1.27 1.27)))
     )
-    (property "Value" "2K" (at 111.76 41.91 90)
+    (property "Value" "5K" (at 111.76 41.91 90)
       (effects (font (size 1.27 1.27)))
     )
@@
   (symbol (lib_id "Device:R_Small") (at 34.925 179.705 270) (unit 1)
     (in_bom yes) (on_board yes) (dnp no) (fields_autoplaced)
-    (property "Reference" "R1" (at 34.925 174.625 90)
-      (effects (font (size 1.27 1.27)))
-    )
-    (property "Value" "10K 5%" (at 34.925 177.165 90)
-      (effects (font (size 1.27 1.27)))
-    )
+    (property "Reference" "R1" (at 34.925 173.99 90)
+      (effects (font (size 1.27 1.27)))
+    )
+    (property "Value" "10K" (at 34.925 176.53 90)
+      (effects (font (size 1.27 1.27)))
+    )
