File: schematic/pcb_v3/pcb_v3.kicad_sch (KiCad schematic)
At the start: 55 parts, among them IC1 FT232RNQ-TRAY, J1 5V, J10 Micro_SD_Card, J2 SERVO, J3 MAVLINK, J4 DISPLAY, J5 SER. SERVO, J6 MAG., J7 U.FL-R, J8 Conn_01x05_Pin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

Commit message: pcb update
Parts:
- removed J10: Micro_SD_Card, symbol Connector:Micro_SD_Card
- added U3: FM24C64B, Package_DFN_QFN:DFN-8_2x2mm_P0.5mm, symbol Memory_NVRAM:FM24C64B
Connections:
- net +3V3: now also U3.8 (VDD)
- net GND: now also U3.4 (VSS), U3.7 (WP)
- net MAG_SCK renamed SCK
- net SCK: now also U3.6 (SCL)
- net MAG_SDI renamed SDI
- net SDI: now also U3.5 (SDA)
- no-connect marks 34 -> 37
Changed lines of the file:
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@@
   (junction (at 152.4 54.61) (diameter 0) (color 0 0 0 0)
   )
+  (junction (at 137.795 173.355) (diameter 0) (color 0 0 0 0)
+  )
   (junction (at 339.09 96.52) (diameter 0) (color 0 0 0 0)
   )
@@
   (no_connect (at 46.355 127.635))
   (no_connect (at 62.865 227.965))
+  (no_connect (at 127.635 165.1))
   (no_connect (at 69.215 120.015))
+  (no_connect (at 127.635 167.64))
   (no_connect (at 220.345 116.84))
   (no_connect (at 46.355 158.115))
@@
   (no_connect (at 215.265 245.745))
   (no_connect (at 215.265 226.695))
+  (no_connect (at 127.635 162.56))
   (no_connect (at 220.345 93.98))
   (no_connect (at 220.345 127))
@@
     (stroke (width 0) (type default))
   )
+  (wire (pts (xy 147.955 162.56) (xy 152.4 162.56))
+    (stroke (width 0) (type default))
+  )
+  (wire (pts (xy 147.955 167.64) (xy 149.86 167.64))
+    (stroke (width 0) (type default))
+  )
   (wire (pts (xy 175.895 207.645) (xy 175.895 222.885))
     (stroke (width 0) (type default))
@@
     (stroke (width 0) (type default))
   )
+  (wire (pts (xy 137.795 173.355) (xy 137.795 172.72))
+    (stroke (width 0) (type default))
+  )
   (wire (pts (xy 277.495 213.36) (xy 281.94 213.36))
     (stroke (width 0) (type default))
@@
     (stroke (width 0) (type default))
   )
+  (wire (pts (xy 137.795 154.305) (xy 137.795 157.48))
+    (stroke (width 0) (type default))
+  )
   (wire (pts (xy 83.185 150.495) (xy 83.185 154.94))
     (stroke (width 0) (type default))
@@
     (stroke (width 0) (type default))
   )
+  (wire (pts (xy 147.955 165.1) (xy 152.4 165.1))
+    (stroke (width 0) (type default))
+  )
   (wire (pts (xy 236.22 217.17) (xy 236.22 222.25))
     (stroke (width 0) (type default))
@@
     (stroke (width 0) (type default))
   )
+  (wire (pts (xy 137.795 174.625) (xy 137.795 173.355))
+    (stroke (width 0) (type default))
+  )
   (wire (pts (xy 289.56 237.49) (xy 289.56 240.665))
     (stroke (width 0) (type default))
@@
     (stroke (width 0) (type default))
   )
+  (wire (pts (xy 149.86 167.64) (xy 149.86 173.355))
+    (stroke (width 0) (type default))
+  )
   (wire (pts (xy 345.44 85.725) (xy 339.09 85.725))
     (stroke (width 0) (type default))
@@
     (stroke (width 0) (type default))
   )
+  (wire (pts (xy 149.86 173.355) (xy 137.795 173.355))
+    (stroke (width 0) (type default))
+  )
   (wire (pts (xy 200.025 272.415) (xy 200.025 274.32))
     (stroke (width 0) (type default))
@@
     )
   )
-  (global_label "MAG_SCK" (shape input) (at 253.365 124.46 0) (fields_autoplaced)
+  (global_label "SCK" (shape input) (at 253.365 124.46 0) (fields_autoplaced)
     (effects (font (size 1.27 1.27)) (justify left))
-    (property "Intersheetrefs" "${INTERSHEET_REFS}" (at 264.8773 124.46 0)
+    (property "Intersheetrefs" "${INTERSHEET_REFS}" (at 260.0997 124.46 0)
       (effects (font (size 1.27 1.27)) (justify left) hide)
     )
@@
     )
   )
-  (global_label "MAG_SDI" (shape input) (at 386.715 203.2 0) (fields_autoplaced)
+  (global_label "SDI" (shape input) (at 386.715 203.2 0) (fields_autoplaced)
     (effects (font (size 1.27 1.27)) (justify left))
-    (property "Intersheetrefs" "${INTERSHEET_REFS}" (at 397.5621 203.2 0)
+    (property "Intersheetrefs" "${INTERSHEET_REFS}" (at 392.7845 203.2 0)
       (effects (font (size 1.27 1.27)) (justify left) hide)
     )
   )
-  (global_label "MAG_SCK" (shape input) (at 386.715 205.74 0) (fields_autoplaced)
+  (global_label "SCK" (shape input) (at 386.715 205.74 0) (fields_autoplaced)
     (effects (font (size 1.27 1.27)) (justify left))
-    (property "Intersheetrefs" "${INTERSHEET_REFS}" (at 398.2273 205.74 0)
+    (property "Intersheetrefs" "${INTERSHEET_REFS}" (at 393.4497 205.74 0)
       (effects (font (size 1.27 1.27)) (justify left) hide)
     )
@@
     )
   )
+  (global_label "SDI" (shape input) (at 152.4 162.56 0) (fields_autoplaced)
+    (effects (font (size 1.27 1.27)) (justify left))
+    (property "Intersheetrefs" "${INTERSHEET_REFS}" (at 158.4695 162.56 0)
+      (effects (font (size 1.27 1.27)) (justify left) hide)
+    )
+  )
   (global_label "VBUS" (shape input) (at 109.855 211.455 180) (fields_autoplaced)
     (effects (font (size 1.27 1.27)) (justify right))
@@
     )
   )
+  (global_label "SCK" (shape input) (at 152.4 165.1 0) (fields_autoplaced)
+    (effects (font (size 1.27 1.27)) (justify left))
+    (property "Intersheetrefs" "${INTERSHEET_REFS}" (at 159.1347 165.1 0)
+      (effects (font (size 1.27 1.27)) (justify left) hide)
+    )
+  )
   (global_label "DTR" (shape input) (at 219.075 221.615 0) (fields_autoplaced)
     (effects (font (size 1.27 1.27)) (justify left))
@@
     )
   )
-  (global_label "MAG_SDI" (shape input) (at 253.365 121.92 0) (fields_autoplaced)
+  (global_label "SDI" (shape input) (at 253.365 121.92 0) (fields_autoplaced)
     (effects (font (size 1.27 1.27)) (justify left))
-    (property "Intersheetrefs" "${INTERSHEET_REFS}" (at 264.2121 121.92 0)
+    (property "Intersheetrefs" "${INTERSHEET_REFS}" (at 259.4345 121.92 0)
       (effects (font (size 1.27 1.27)) (justify left) hide)
     )
@@
     )
   )
+  (symbol (lib_id "power:GND") (at 137.795 174.625 0) (unit 1)
+    (in_bom yes) (on_board yes) (dnp no) (fields_autoplaced)
+    (property "Reference" "#PWR010" (at 137.795 180.975 0)
+      (effects (font (size 1.27 1.27)) hide)
+    )
+    (property "Value" "GND" (at 137.795 178.943 0)
+      (effects (font (size 1.27 1.27)))
+    )
+    (property "Footprint" "" (at 137.795 174.625 0)
+      (effects (font (size 1.27 1.27)) hide)
+    )
+    (property "Datasheet" "" (at 137.795 174.625 0)
+      (effects (font (size 1.27 1.27)) hide)
+    )
+    (pin "1")
+    (instances
+      (project "pcb_v3"
+        (path "/b282be2a-417a-4cfb-98a6-eaf74523d760"
+          (reference "#PWR010") (unit 1)
+        )
+      )
+      (project "pcb"
+        (path "/bb09d15e-8949-465f-96ce-de682ac5520f"
+          (reference "#PWR016") (unit 1)
+        )
+      )
+    )
+  )
   (symbol (lib_id "Device:R_Small") (at 334.01 46.355 0) (unit 1)
     (in_bom yes) (on_board yes) (dnp no) (fields_autoplaced)
@@
     )
   )
+  (symbol (lib_id "power:+3V3") (at 137.795 154.305 0) (unit 1)
+    (in_bom yes) (on_board yes) (dnp no) (fields_autoplaced)
+    (property "Reference" "#PWR034" (at 137.795 158.115 0)
+      (effects (font (size 1.27 1.27)) hide)
+    )
+    (property "Value" "+3V3" (at 137.795 149.479 0)
+      (effects (font (size 1.27 1.27)))
+    )
+    (property "Footprint" "" (at 137.795 154.305 0)
+      (effects (font (size 1.27 1.27)) hide)
+    )
+    (property "Datasheet" "" (at 137.795 154.305 0)
+      (effects (font (size 1.27 1.27)) hide)
+    )
+    (pin "1")
+    (instances
+      (project "pcb_v3"
+        (path "/b282be2a-417a-4cfb-98a6-eaf74523d760"
+          (reference "#PWR034") (unit 1)
+        )
+      )
+      (project "pcb"
+        (path "/bb09d15e-8949-465f-96ce-de682ac5520f"
+          (reference "#PWR028") (unit 1)
+        )
+      )
+    )
+  )
   (symbol (lib_id "RF_Module:ESP32-WROOM-32") (at 235.585 116.84 0) (unit 1)
     (in_bom yes) (on_board yes) (dnp no) (fields_autoplaced)
@@
     )
   )
+  (symbol (lib_id "Memory_NVRAM:FM24C64B") (at 137.795 165.1 0) (unit 1)
+    (in_bom yes) (on_board yes) (dnp no) (fields_autoplaced)
+    (property "Reference" "U3" (at 139.9891 154.94 0)
+      (effects (font (size 1.27 1.27)) (justify left))
+    )
+    (property "Value" "FM24C64B" (at 139.9891 157.48 0)
+      (effects (font (size 1.27 1.27)) (justify left))
+    )
+    (property "Footprint" "Package_DFN_QFN:DFN-8_2x2mm_P0.5mm" (at 137.795 153.67 0)
+      (effects (font (size 1.27 1.27)) hide)
+    )
+    (property "Datasheet" "http://www.cypress.com/file/41651/download" (at 137.795 151.13 0)
+      (effects (font (size 1.27 1.27)) hide)
+    )
+    (pin "1")
+    (pin "2")
+    (pin "3")
+    (pin "4")
+    (pin "5")
+    (pin "6")
+    (pin "7")
+    (pin "8")
+    (instances
+      (project "pcb_v3"
+        (path "/b282be2a-417a-4cfb-98a6-eaf74523d760"
+          (reference "U3") (unit 1)
+        )
+      )
+    )
+  )
   (symbol (lib_id "power:GND") (at 64.135 117.475 180) (unit 1)
     (in_bom yes) (on_board yes) (dnp no) (fields_autoplaced)
@@
         )
       )
-    )
-  )
-  (symbol (lib_id "Connector:Micro_SD_Card") (at 272.415 43.18 0) (unit 1)
-    (in_bom yes) (on_board yes) (dnp no) (fields_autoplaced)
-    (property "Reference" "J10" (at 273.05 24.765 0)
-      (effects (font (size 1.27 1.27)))
-    )
-    (property "Value" "Micro_SD_Card" (at 273.05 27.305 0)
-      (effects (font (size 1.27 1.27)))
-    )
-    (property "Footprint" "" (at 301.625 35.56 0)
-      (effects (font (size 1.27 1.27)) hide)
-    )
-    (property "Datasheet" "http://katalog.we-online.de/em/datasheet/693072010801.pdf" (at 272.415 43.18 0)
-      (effects (font (size 1.27 1.27)) hide)
-    )
-    (pin "1")
-    (pin "2")
-    (pin "3")
-    (pin "4")
-    (pin "5")
-    (pin "6")
-    (pin "7")
-    (pin "8")
-    (pin "9")
-    (instances
-      (project "pcb_v3"
-        (path "/b282be2a-417a-4cfb-98a6-eaf74523d760"
-          (reference "J10") (unit 1)
-        )
-      )

Commit message: fram, gps uart
Parts:
- added J10: UART/SPI, Connector_PinHeader_2.54mm:PinHeader_1x02_P2.54mm_Vertical, symbol Connector:Conn_01x02_Pin
- added J11: Conn_01x03_Pin, Connector_PinHeader_2.54mm:PinHeader_1x03_P2.54mm_Vertical, symbol Connector:Conn_01x03_Pin
- added R12, R13: 2.2K, Resistor_SMD:R_0805_2012Metric, symbol Device:R_Small
Connections:
- net +3V3: now also R12.1, R13.1
- net +5V: now also J2.2 (Pin_2); no longer J2.3 (Pin_3)
- net GND: now also U3.1 (A0), U3.2 (A1), U3.3 (A2), J10.2 (Pin_2), J11.1 (Pin_1); no longer U1.2 (D_SEL)
- net SCK: now also R12.2
- net SDI: now also R13.2
- net SERVO: now also J2.3 (Pin_3); no longer J2.2 (Pin_2)
- net GPS_MISO renamed GPS_MISO/TX
- net GPS_MISO/TX: now also J11.3 (Pin_3)
- net GPS_MOSI renamed GPS_MOSI/RX
- net GPS_MOSI/RX: now also J11.2 (Pin_2)
- new net: J10.1 (Pin_1), U1.2 (D_SEL)
- no-connect marks 37 -> 34

Commit message: pcb cleanup
Other:
- moved on the sheet: C10, C12, C9, D3, ESP1, R10, R12, R13, R9, U3

Commit message: final pcb please
Parts:
- added TP1: TestPoint, TestPoint:TestPoint_Pad_D1.5mm, symbol Connector:TestPoint
Connections:
- net GND: no longer U3.1 (A0)
- new net: TP1.1, U3.1 (A0)
Changed lines of the file:
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@@
   (junction (at 36.83 120.65) (diameter 0) (color 0 0 0 0)
   )
-  (junction (at 137.795 166.37) (diameter 0) (color 0 0 0 0)
-  )
   (junction (at 215.9 59.69) (diameter 0) (color 0 0 0 0)
   )
@@
     (stroke (width 0) (type default))
   )
-  (wire (pts (xy 137.795 166.37) (xy 137.795 163.83))
-    (stroke (width 0) (type default))
-  )
   (wire (pts (xy 384.81 203.2) (xy 386.715 203.2))
     (stroke (width 0) (type default))
@@
         )
       )
+    )
+  )
+  (symbol (lib_id "Connector:TestPoint") (at 137.795 163.83 90) (unit 1)
+    (in_bom yes) (on_board yes) (dnp no) (fields_autoplaced)
+    (property "Reference" "TP1" (at 134.493 158.75 90)
+      (effects (font (size 1.27 1.27)))
+    )
+    (property "Value" "TestPoint" (at 134.493 161.29 90)
+      (effects (font (size 1.27 1.27)))
+    )
+    (property "Footprint" "TestPoint:TestPoint_Pad_D1.5mm" (at 137.795 158.75 0)
+      (effects (font (size 1.27 1.27)) hide)
+    )
+    (property "Datasheet" "~" (at 137.795 158.75 0)
+      (effects (font (size 1.27 1.27)) hide)
+    )
+    (pin "1")
+    (instances
+      (project "pcb_v3"
+        (path "/b282be2a-417a-4cfb-98a6-eaf74523d760"
+          (reference "TP1") (unit 1)
+        )
+      )

Commit message: magnetometer interface, cleanup
Parts:
- removed TP1: TestPoint, TestPoint:TestPoint_Pad_D1.5mm, symbol Connector:TestPoint
- U3: footprint Package_DFN_QFN:DFN-8_2x2mm_P0.5mm -> Package_SON:SON95P400X450X80-9N
Connections:
- net GND: no longer U3.2 (A1), U3.3 (A2)
- no-connect marks 34 -> 37
Changed lines of the file:
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@@
   (junction (at 326.39 40.64) (diameter 0) (color 0 0 0 0)
   )
-  (junction (at 137.795 168.91) (diameter 0) (color 0 0 0 0)
-  )
   (junction (at 187.96 53.975) (diameter 0) (color 0 0 0 0)
   )
@@
   (no_connect (at 179.705 243.205))
   (no_connect (at 179.705 229.235))
+  (no_connect (at 140.335 166.37))
   (no_connect (at 46.355 155.575))
   (no_connect (at 215.265 224.155))
@@
   (no_connect (at 215.265 259.715))
   (no_connect (at 215.265 245.745))
+  (no_connect (at 140.335 168.91))
   (no_connect (at 215.265 226.695))
   (no_connect (at 220.345 78.105))
@@
   (no_connect (at 215.265 240.665))
   (no_connect (at 215.265 243.205))
+  (no_connect (at 140.335 163.83))
   (no_connect (at 46.355 130.175))
   (no_connect (at 179.705 234.315))
@@
     (stroke (width 0) (type default))
   )
-  (wire (pts (xy 137.795 174.625) (xy 137.795 168.91))
-    (stroke (width 0) (type default))
-  )
-  (wire (pts (xy 137.795 168.91) (xy 137.795 166.37))
-    (stroke (width 0) (type default))
-  )
   (wire (pts (xy 289.56 218.44) (xy 289.56 219.71))
     (stroke (width 0) (type default))
@@
     (stroke (width 0) (type default))
   )
-  (wire (pts (xy 137.795 163.83) (xy 140.335 163.83))
-    (stroke (width 0) (type default))
-  )
   (wire (pts (xy 175.895 110.49) (xy 184.15 110.49))
     (stroke (width 0) (type default))
@@
     (stroke (width 0) (type default))
   )
-  (wire (pts (xy 137.795 166.37) (xy 140.335 166.37))
-    (stroke (width 0) (type default))
-  )
   (wire (pts (xy 46.99 113.03) (xy 36.83 113.03))
     (stroke (width 0) (type default))
@@
     (stroke (width 0) (type default))
   )
-  (wire (pts (xy 137.795 168.91) (xy 140.335 168.91))
-    (stroke (width 0) (type default))
-  )
   (wire (pts (xy 162.56 255.905) (xy 179.705 255.905))
     (stroke (width 0) (type default))
@@
     (stroke (width 0) (type default))
   )
-  (wire (pts (xy 150.495 174.625) (xy 137.795 174.625))
-    (stroke (width 0) (type default))
-  )
   (wire (pts (xy 250.825 128.905) (xy 252.73 128.905))
     (stroke (width 0) (type default))
@@
     )
   )
-  (symbol (lib_id "Connector:TestPoint") (at 137.795 163.83 90) (unit 1)
-    (in_bom yes) (on_board yes) (dnp no) (fields_autoplaced)
-    (property "Reference" "TP1" (at 134.493 158.75 90)
-      (effects (font (size 1.27 1.27)))
-    )
-    (property "Value" "TestPoint" (at 134.493 161.29 90)
-      (effects (font (size 1.27 1.27)))
-    )
-    (property "Footprint" "TestPoint:TestPoint_Pad_D1.5mm" (at 137.795 158.75 0)
-      (effects (font (size 1.27 1.27)) hide)
-    )
-    (property "Datasheet" "~" (at 137.795 158.75 0)
-      (effects (font (size 1.27 1.27)) hide)
-    )
-    (pin "1")
-    (instances
-      (project "pcb_v3"
-        (path "/b282be2a-417a-4cfb-98a6-eaf74523d760"
-          (reference "TP1") (unit 1)
-        )
-      )
-    )
-  )
   (symbol (lib_id "Connector:Conn_01x03_Pin") (at 379.73 224.79 0) (unit 1)
     (in_bom yes) (on_board yes) (dnp no) (fields_autoplaced)
@@
       (effects (font (size 1.27 1.27)) (justify left))
     )
-    (property "Footprint" "Package_DFN_QFN:DFN-8_2x2mm_P0.5mm" (at 150.495 154.94 0)
+    (property "Footprint" "Package_SON:SON95P400X450X80-9N" (at 150.495 154.94 0)
       (effects (font (size 1.27 1.27)) hide)
     )

Commit message: tests
Parts:
- added C16: 100nF, Capacitor_SMD:C_0805_2012Metric, symbol Device:C_Small
- added L1: 27nH, Inductor_SMD:L_0805_2012Metric, symbol Device:L_Small
- added R14: 20, Resistor_SMD:R_0805_2012Metric, symbol Device:R_Small
Connections:
- net GND: now also C16.1
- net at J7.2, U1.11 (RF_IN): now also L1.2
- net at U1.9 (VCC_RF): now also R14.1
- new net: C16.2, L1.1, R14.2
- no-connect marks 37 -> 36
Other:
- moved on the sheet: J7
