File: schematic/pcb_v3/pcb_v3.kicad_pcb (KiCad board)
At the start: 4 copper layers, 56 x 56 mm, 66 parts, among them IC1 FT232RNQ-TRAY, J1 5V, J10 UART/SPI, J11 Conn_01x03_Pin, J2 SERVO, J3 MAVLINK, J4 DISPLAY, J5 SER. SERVO, J6 MAG., J7 U.FL-R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

Commit message: correct heartbeat, misc
Parts:
- added REF**: MountingHole_2.2mm_M2_ISO7380_Pad, MountingHole:MountingHole_2.2mm_M2_ISO7380_Pad, F.Cu at (239.8, 110.9)
- added REF**: MountingHole_2.2mm_M2_ISO7380_Pad, MountingHole:MountingHole_2.2mm_M2_ISO7380_Pad, F.Cu at (189.8, 110.9)
- J8: moved to B.Cu
- moved SW5 241.8 mm to (231.9, 110.9)
- moved SW4 234.1 mm to (220.4, 110.9)
- moved J8 227.8 mm to (214.8, 110.6), turned to -90 degrees
- moved SW3 227.4 mm to (209.3, 110.9)
- moved SW2 221.0 mm to (197.8, 110.9)
Routing:
- net BUTTON_1: track 0.00 -> 22.6 mm, vias 0 -> 1
- net BUTTON_4: track 0.00 -> 21.4 mm, vias 0 -> 1
- net BUTTON_3: track 0.00 -> 15.3 mm, vias 0 -> 1
- net BUTTON_2: track 0.00 -> 9.86 mm, vias 0 -> 1
- net GND1: track 0.00 -> 2.35 mm, vias 0 -> 1
- added copper zone on B.Cu, net GND1
- added copper zone on F.Cu, net GND1
Other:
- board size 56 x 56 mm -> 56.2 x 69.9 mm
- board text added: "BUTTON 1"
- board text added: "BUTTON 2"
- board text added: "BUTTON 3"
- board text added: "BUTTON 4"
